File: hardware/LeftConnector/LeftConnector.kicad_sch (KiCad schematic)
At the start: 3 parts, among them J1 Conn_01x10, J2 Conn_01x10

Commit message: Left connector initial FPC
Parts:
- C1: footprint consolizer:flex_long_10 -> consolizer:flex_short_10
Changed lines of the file:
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@@
       (effects (font (size 1.27 1.27)) (justify left))
     )
-    (property "Footprint" "consolizer:flex_long_10" (id 2) (at 102.87 66.04 0)
+    (property "Footprint" "consolizer:flex_short_10" (id 2) (at 102.87 66.04 0)
       (effects (font (size 1.27 1.27)) hide)
     )
@@
   (symbol_instances
     (path "/ea6fde00-59dc-4a79-a647-7e38199fae0e"
-      (reference "C1") (unit 1) (value "trill-flex-conector_10") (footprint "consolizer:flex_long_10")
+      (reference "C1") (unit 1) (value "trill-flex-conector_10") (footprint "consolizer:flex_short_10")
     )
     (path "/a07b6b2b-7179-4297-b163-5e47ffbe76d3"
