File: hardware/CenterConnecto/CenterConnecto.kicad_sch (KiCad schematic)
At the start: 3 parts, among them J1 Conn_01x10, J2 Conn_01x10

Commit message: Added initial left buttons fpc
Parts:
- C1: footprint consolizer:flex_long_10 -> consolizer:flex_short_10
Changed lines of the file:
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@@
       (effects (font (size 1.27 1.27)) (justify left))
     )
-    (property "Footprint" "consolizer:flex_long_10" (id 2) (at 77.47 78.74 0)
+    (property "Footprint" "consolizer:flex_short_10" (id 2) (at 77.47 78.74 0)
       (effects (font (size 1.27 1.27)) hide)
     )
@@
   (symbol_instances
     (path "/0fe459be-6237-4e69-9849-b12b113e8605"
-      (reference "C1") (unit 1) (value "trill-flex-conector_10") (footprint "consolizer:flex_long_10")
+      (reference "C1") (unit 1) (value "trill-flex-conector_10") (footprint "consolizer:flex_short_10")
     )
     (path "/2e586240-f606-4214-a0bb-6944933b64f5"
