File: hardware/lbuttons/lbuttons.kicad_pcb (KiCad board)
At the start: 2 copper layers, 39.4 x 55 mm, 11 parts, among them J1 Conn_01x01, J2 Conn_01x01, J3 Conn_01x01, J4 Conn_01x01, J5 Conn_01x01, SW1 SKQGADE010, SW2 SKQGADE010, SW3 SKQGADE010, SW4 SKQGADE010, SW5 SKQGADE010

Commit message: Cleanup and add documentation
Parts:
- removed C1: trill-flex-conector_10, consolizer:flex_short_10
- removed J1, J2, J3, J4, J5: Conn_01x01, TestPoint:TestPoint_Pad_1.0x1.0mm
- removed SW1, SW2, SW3, SW4, SW5: SKQGADE010, JLCPCB_footprint:SW-SMD_4P-L5.2-W5.2-P3.70-LS6.4
- added C3: flex-conector_10, consolizer:flex_short_10, F.Cu at (148.5, 123.2)
- added C4: flex-conector_10, consolizer:flex_short_10, F.Cu at (220.5, 133.5)
- added U1: SKRBAKE010, JLCPCB_footprint:KEY-SMD_4P-L4.0-W4.8-P3.90-LS4.8, F.Cu at (122.8, 87.0)
- added U2: SKRBAKE010, JLCPCB_footprint:KEY-SMD_4P-L4.0-W4.8-P3.90-LS4.8, F.Cu at (132.0, 115.5)
- added U3: SKRBAKE010, JLCPCB_footprint:KEY-SMD_4P-L4.0-W4.8-P3.90-LS4.8, F.Cu at (124.5, 108.0)
- added U4: SKRBAKE010, JLCPCB_footprint:KEY-SMD_4P-L4.0-W4.8-P3.90-LS4.8, F.Cu at (117.0, 115.5)
- added U5: SKRBAKE010, JLCPCB_footprint:KEY-SMD_4P-L4.0-W4.8-P3.90-LS4.8, F.Cu at (124.5, 123.0)
Routing:
- net GND: track 127.8 -> 257.8 mm, vias 0 -> 2
- net /down: track 59.8 -> 134.5 mm, vias 0 -> 4
- net /right: track 55.4 -> 124.8 mm, vias 0 -> 2
- net /left: track 74.4 -> 142.1 mm, vias 0 -> 4
- net /up: track 74.9 -> 142.4 mm, vias 0 -> 4
- net /l1: track 128.6 -> 158.1 mm, vias 0 -> 2
Other:
- board size 39.4 x 55 mm -> 107.7 x 55 mm
- board text added: "PSP"

Commit message: Latest
Parts:
- removed U1, U2, U3, U4, U5: SKRBAKE010, JLCPCB_footprint:KEY-SMD_4P-L4.0-W4.8-P3.90-LS4.8
- added DOWN1: K2-1187SQ-E4SW-06, JLCPCB_footprint:KEY-SMD_4P-L5.2-W5.2-P3.70-LS6.4, F.Cu at (91.1, 122.2)
- added L1: K2-1187SQ-E4SW-06, JLCPCB_footprint:KEY-SMD_4P-L5.2-W5.2-P3.70-LS6.4, F.Cu at (89.4, 86.2)
- added LEFT1: K2-1187SQ-E4SW-06, JLCPCB_footprint:KEY-SMD_4P-L5.2-W5.2-P3.70-LS6.4, F.Cu at (83.6, 114.8)
- added RIGHT1: K2-1187SQ-E4SW-06, JLCPCB_footprint:KEY-SMD_4P-L5.2-W5.2-P3.70-LS6.4, F.Cu at (98.6, 114.8)
- added UP1: K2-1187SQ-E4SW-06, JLCPCB_footprint:KEY-SMD_4P-L5.2-W5.2-P3.70-LS6.4, F.Cu at (91.1, 107.2)
- moved C3 33.4 mm to (115.1, 122.5)
- moved C4 18.4 mm to (202.1, 132.8)
Routing:
- net GND: track 257.8 -> 333.8 mm, vias 2 -> 5
- net /left: track 142.1 -> 160.6 mm, vias 4 -> 2
- net /up: track 142.4 -> 159.3 mm, vias 4 -> 2
- net /l1: track 158.1 -> 170.3 mm
- net /right: track 124.8 -> 136.3 mm
- net /down: track 134.5 -> 144.2 mm, vias 4 -> 2
Other:
- board size 107.7 x 55 mm -> 122.7 x 55 mm
- board text added: "A"
