File: hardware/lbuttons/lbuttons.kicad_sch (KiCad schematic)
At the start: 11 parts, among them J1 Conn_01x01, J2 Conn_01x01, J3 Conn_01x01, J4 Conn_01x01, J5 Conn_01x01, SW1 SKQGADE010, SW2 SKQGADE010, SW3 SKQGADE010, SW4 SKQGADE010, SW5 SKQGADE010

Commit message: Cleanup and add documentation
Parts:
- removed C1: trill-flex-conector_10, consolizer:flex_short_10, symbol consolizer:trill-flex-conector_10
- removed J1, J2, J3, J4, J5: Conn_01x01, TestPoint:TestPoint_Pad_1.0x1.0mm, symbol Connector_Generic:Conn_01x01
- removed SW1, SW2, SW3, SW4, SW5: SKQGADE010, JLCPCB_footprint:SW-SMD_4P-L5.2-W5.2-P3.70-LS6.4, symbol JLCPCB_schematic:SKQGADE010
- added C3, C4: flex-conector_10, consolizer:flex_short_10, symbol consolizer:flex-conector_10
- added U1, U2, U3, U4, U5: SKRBAKE010, JLCPCB_footprint:KEY-SMD_4P-L4.0-W4.8-P3.90-LS4.8, symbol JLCPCB_schematic:SKRBAKE010
Connections:
- net GND: now also C3.10, C3.6, C3.7, C3.8, C3.9, C4.10, C4.6, C4.7, C4.8, C4.9, U1.2, U1.4, U2.2, U2.4, U3.2, U3.4, U4.2, U4.4, U5.2, U5.4
- net down: now also C3.5, C4.5, U5.1, U5.3
- net l1: now also C3.1, C4.1, U1.1, U1.3
- net left: now also C3.4, C4.4, U4.1, U4.3
- net right: now also C3.2, C4.2, U2.1, U2.3
- net up: now also C3.3, C4.3, U3.1, U3.3

Commit message: Latest
Parts:
- removed U1, U2, U3, U4, U5: SKRBAKE010, JLCPCB_footprint:KEY-SMD_4P-L4.0-W4.8-P3.90-LS4.8, symbol JLCPCB_schematic:SKRBAKE010
- added DOWN1, L1, LEFT1, RIGHT1, UP1: K2-1187SQ-E4SW-06, JLCPCB_footprint:KEY-SMD_4P-L5.2-W5.2-P3.70-LS6.4, symbol JLCPCB_schematic:K2-1187SQ-E4SW-06
Connections:
- net GND: now also DOWN1.3, DOWN1.4, L1.3, L1.4, LEFT1.3, LEFT1.4, RIGHT1.3, RIGHT1.4, UP1.3, UP1.4
- net down: now also DOWN1.1, DOWN1.2
- net l1: now also L1.1, L1.2
- net left: now also LEFT1.1, LEFT1.2
- net right: now also RIGHT1.1, RIGHT1.2
- net up: now also UP1.1, UP1.2
Other:
- moved on the sheet: C3, C4
