File: hardware/rbuttons/rbuttons.kicad_sch (KiCad schematic)
At the start: 8 parts, among them U1 SKRBAKE010, U2 SKRBAKE010, U3 SKRBAKE010, U4 SKRBAKE010, U5 SKRBAKE010

Commit message: Latest
Parts:
- removed U1, U2, U3, U4, U5: SKRBAKE010, JLCPCB_footprint:KEY-SMD_4P-L4.0-W4.8-P3.90-LS4.8, symbol JLCPCB_schematic:SKRBAKE010
- added CIRCLE1, CROSS1, R1, SQUARE1, TRIANGLE1: K2-1187SQ-E4SW-06, JLCPCB_footprint:KEY-SMD_4P-L5.2-W5.2-P3.70-LS6.4, symbol JLCPCB_schematic:K2-1187SQ-E4SW-06
Connections:
- net Circle: now also C1.11, CIRCLE1.1, CIRCLE1.2; no longer C1.4
- net R1: now also C1.13, R1.1, R1.2; no longer C1.2
- net Square: now also C1.14, SQUARE1.1, SQUARE1.2; no longer C1.1
- net Triangle: now also C1.12, TRIANGLE1.1, TRIANGLE1.2; no longer C1.3
- net cross: now also C1.10, CROSS1.1, CROSS1.2; no longer C1.5
- net five: now also C1.1, C2.7; no longer C1.14, C2.2
- net four: now also C1.2, C2.6; no longer C1.13, C2.3
- net gnd: now also C2.1, C2.2, CIRCLE1.3, CIRCLE1.4, CROSS1.3, CROSS1.4, R1.3, R1.4, SQUARE1.3, SQUARE1.4, TRIANGLE1.3, TRIANGLE1.4; no longer C2.7, C2.8
- net one: now also C1.5, C2.3; no longer C1.10, C2.6
- net three: now also C1.3, C2.5; no longer C1.12, C2.4
- net tw: now also C1.4, C2.4; no longer C1.11, C2.5
